Commit message: dont think this works but ill dump it here

File: TestSite/ws_rviz/src/ur3e_workstation/urdf/workstation.xacro (robot description, xacro)
@@ -11,4 +11,5 @@
   <xacro:arg name="output_recipe_filename" default=""/>
   <xacro:arg name="input_recipe_filename" default=""/>
+  <xacro:arg name="base_at_world_origin" default="false"/>
   <!-- ==================== World ==================== -->
   <link name="world"/>
@@ -55,13 +56,24 @@
   <!-- ==================== UR3e Robot ==================== -->
   <xacro:include filename="$(find ur_description)/urdf/ur_macro.xacro"/>
+  <!-- Select robot parent and pose based on base_at_world_origin -->
+  <xacro:if value="$(arg base_at_world_origin)">
+    <xacro:property name="robot_parent" value="world"/>
+    <xacro:property name="robot_xyz" value="0 0 0"/>
+    <xacro:property name="robot_rpy" value="0 0 0"/>
+  </xacro:if>
+  <xacro:unless value="$(arg base_at_world_origin)">
+    <xacro:property name="robot_parent" value="mount"/>
+    <xacro:property name="robot_xyz" value="0 -0.218 0"/>
+    <xacro:property name="robot_rpy" value="-1.5708 0 3.1416"/>
+  </xacro:unless>
   <xacro:ur_robot
     name="$(arg ur_type)"
     tf_prefix=""
-    parent="mount"
+    parent="${robot_parent}"
     joint_limits_parameters_file="$(find ur_description)/config/$(arg ur_type)/joint_limits.yaml"
     kinematics_parameters_file="$(find ur_description)/config/$(arg ur_type)/default_kinematics.yaml"
     physical_parameters_file="$(find ur_description)/config/$(arg ur_type)/physical_parameters.yaml"
     visual_parameters_file="$(find ur_description)/config/$(arg ur_type)/visual_parameters.yaml">
-    <origin xyz="0 -0.218 0" rpy="-1.5708 0 3.1416"/>
+    <origin xyz="${robot_xyz}" rpy="${robot_rpy}"/>
   </xacro:ur_robot>
   <!-- Add ros2_control for the UR robot -->

File: TestSite/ws_rviz/src/ur3e_workstation/urdf/workstation_with_ros2_control.xacro (robot description, xacro)
@@ -1,139 +1,104 @@
 <?xml version="1.0"?>
-<robot xmlns:xacro="http://www.ros.org/wiki/xacro" name="ur3e_workstation">
-  <!-- Arguments -->
-  <xacro:arg name="ur_type" default="ur3e"/>
-  <xacro:arg name="robot_ip" default="192.168.56.101"/>
-  <xacro:arg name="use_mock_hardware" default="true"/>
-  <xacro:arg name="mock_sensor_commands" default="false"/>
-  <xacro:arg name="headless_mode" default="false"/>
-  <xacro:arg name="initial_positions_file" default="$(find ur_description)/config/initial_positions.yaml"/>
-  <xacro:arg name="script_filename" default=""/>
-  <xacro:arg name="output_recipe_filename" default=""/>
-  <xacro:arg name="input_recipe_filename" default=""/>
-  <!-- ==================== World ==================== -->
-  <link name="world"/>
-  <!-- ==================== Table / Bordplade ==================== -->
-  <link name="bordplade">
-    <visual>
-      <geometry>
-        <mesh filename="package://ur3e_workstation/urdf/Bundplade.stl" scale="0.001 0.001 0.001"/>
-      </geometry>
-      <origin xyz="0 0 0" rpy="0 0 0"/>
-    </visual>
-    <collision>
-      <geometry>
-        <mesh filename="package://ur3e_workstation/urdf/Bundplade.stl" scale="0.001 0.001 0.001"/>
-      </geometry>
-      <origin xyz="0 0 0" rpy="0 0 0"/>
-    </collision>
-  </link>
-  <joint name="world_to_bordplade" type="fixed">
-    <parent link="world"/>
-    <child link="bordplade"/>
-    <origin xyz="0 0 0" rpy="0 0 0"/>
-  </joint>
-  <!-- ==================== Mount ==================== -->
-  <link name="mount">
-    <visual>
-      <geometry>
-        <mesh filename="package://ur3e_workstation/urdf/UR3e_mount.stl" scale="0.001 0.001 0.001"/>
-      </geometry>
-      <origin xyz="0 0 0" rpy="0 0 0"/>
-    </visual>
-    <collision>
-      <geometry>
-        <mesh filename="package://ur3e_workstation/urdf/UR3e_mount.stl" scale="0.001 0.001 0.001"/>
-      </geometry>
-      <origin xyz="0 0 0" rpy="0 0 0"/>
-    </collision>
-  </link>
-  <joint name="bordplade_to_mount" type="fixed">
-    <parent link="bordplade"/>
-    <child link="mount"/>
-    <origin xyz="0.200 0.0 0.250" rpy="0 0 0"/>
-  </joint>
-  <!-- ==================== UR3e Robot with ros2_control ==================== -->
+<robot xmlns:xacro="http://www.ros.org/wiki/xacro">
+  <!-- Include UR description macros -->
   <xacro:include filename="$(find ur_description)/urdf/ur_macro.xacro"/>
-  <xacro:ur_robot
-    name="$(arg ur_type)"
-    tf_prefix=""
-    parent="mount"
-    joint_limits_parameters_file="$(find ur_description)/config/$(arg ur_type)/joint_limits.yaml"
-    kinematics_parameters_file="$(find ur_description)/config/$(arg ur_type)/default_kinematics.yaml"
-    physical_parameters_file="$(find ur_description)/config/$(arg ur_type)/physical_parameters.yaml"
-    visual_parameters_file="$(find ur_description)/config/$(arg ur_type)/visual_parameters.yaml"
-    transmission_hw_interface="hardware_interface/PositionJointInterface"
-    safety_limits="false"
-    safety_pos_margin="0.15"
-    safety_k_position="20"
-    use_mock_hardware="$(arg use_mock_hardware)"
-    mock_sensor_commands="$(arg mock_sensor_commands)"
-    headless_mode="$(arg headless_mode)"
-    robot_ip="$(arg robot_ip)"
-    script_filename="$(arg script_filename)"
-    output_recipe_filename="$(arg output_recipe_filename)"
-    input_recipe_filename="$(arg input_recipe_filename)"
-    initial_positions_file="$(arg initial_positions_file)">
-    <origin xyz="0 -0.218 0" rpy="-1.5708 0 3.1416"/>
-  </xacro:ur_robot>
-  <!-- ==================== Test Plate ==================== -->
-  <link name="testpladekurve">
-    <visual>
-      <geometry>
-        <mesh filename="package://ur3e_workstation/urdf/TestpladeKurve_v3.stl" scale="0.001 0.001 0.001"/>
-      </geometry>
-      <origin xyz="0.200 2.94 -0.4" rpy="1.5708 0 0"/>
-    </visual>
-    <collision>
-      <geometry>
-        <mesh filename="package://ur3e_workstation/urdf/TestpladeKurve_v3.stl" scale="0.001 0.001 0.001"/>
-      </geometry>
-      <origin xyz="0.200 0 0" rpy="1.5708 0 0"/>
-    </collision>
-  </link>
-  <joint name="bordplade_to_testpladekurve" type="fixed">
-    <parent link="bordplade"/>
-    <child link="testpladekurve"/>
-    <origin xyz="0 0 0" rpy="0 0 0"/>
-  </joint>
-  <!-- ==================== Realsense Holder ==================== -->
-  <link name="realsense_holder">
-    <visual>
-      <geometry>
-        <mesh filename="package://ur3e_workstation/urdf/RealsenseHolder.stl" scale="0.001 0.001 0.001"/>
-      </geometry>
-      <origin xyz="0 0 0" rpy="0 0 0"/>
-    </visual>
-    <collision>
-      <geometry>
-        <mesh filename="package://ur3e_workstation/urdf/RealsenseHolder.stl" scale="0.001 0.001 0.001"/>
-      </geometry>
-      <origin xyz="0 0 0" rpy="0 0 0"/>
-    </collision>
-  </link>
-  <joint name="ee_to_holder" type="fixed">
-    <parent link="tool0"/>
-    <child link="realsense_holder"/>
-    <origin xyz="0 0 -0.085" rpy="0 0 0"/>
-  </joint>
-  <!-- ==================== RSD435 Camera ==================== -->
-  <link name="rsd435">
-    <visual>
-      <geometry>
-        <mesh filename="package://ur3e_workstation/urdf/RSD435.stl" scale="0.001 0.001 0.001"/>
-      </geometry>
-      <origin xyz="0 0 0" rpy="0 0 0"/>
-    </visual>
-    <collision>
-      <geometry>
-        <mesh filename="package://ur3e_workstation/urdf/RSD435.stl" scale="0.001 0.001 0.001"/>
-      </geometry>
-      <origin xyz="0 0 0" rpy="0 0 0"/>
-    </collision>
-  </link>
-  <joint name="holder_to_camera" type="fixed">
-    <parent link="realsense_holder"/>
-    <child link="rsd435"/>
-    <origin xyz="0 0.044 0.072" rpy="0 0 0"/>
-  </joint>
+  <!--
+    Updated macro that mimics the workstation-style UR3e setup.
+    It expects arguments similar to the second file.
+  -->
+  <xacro:macro
+    name="my_robot_cell"
+    params="
+      parent
+      *origin
+      ur_type
+      robot_ip
+      use_mock_hardware
+      mock_sensor_commands
+      headless_mode
+      initial_positions_file
+      script_filename
+      output_recipe_filename
+      input_recipe_filename
+      base_at_world_origin
+    ">
+    <!-- ==================== BASE LINK / TABLE ==================== -->
+    <joint name="world_to_bordplade" type="fixed">
+      <xacro:insert_block name="origin" />
+      <parent link="${parent}"/>
+      <child link="bordplade"/>
+    </joint>
+    <link name="bordplade">
+      <visual>
+        <geometry>
+          <mesh filename="package://my_robot_cell_description/meshes/Bundplade.stl"
+                scale="0.001 0.001 0.001"/>
+        </geometry>
+      </visual>
+      <collision>
+        <geometry>
+          <mesh filename="package://my_robot_cell_description/meshes/Bundplade.stl"
+                scale="0.001 0.001 0.001"/>
+        </geometry>
+      </collision>
+    </link>
+    <!-- ==================== MOUNT ==================== -->
+    <link name="mount">
+      <visual>
+        <geometry>
+          <mesh filename="package://my_robot_cell_description/meshes/UR3e_mount.stl"
+                scale="0.001 0.001 0.001"/>
+        </geometry>
+      </visual>
+      <collision>
+        <geometry>
+          <mesh filename="package://my_robot_cell_description/meshes/UR3e_mount.stl"
+                scale="0.001 0.001 0.001"/>
+        </geometry>
+      </collision>
+    </link>
+    <joint name="bordplade_to_mount" type="fixed">
+      <parent link="bordplade"/>
+      <child link="mount"/>
+      <origin xyz="0.200 0.0 0.250" rpy="0 0 0"/>
+    </joint>
+    <!-- ==================== Robot Parent Logic ==================== -->
+    <xacro:if value="${base_at_world_origin}">
+      <xacro:property name="robot_parent" value="${parent}"/>
+      <xacro:property name="robot_xyz"    value="0 0 0"/>
+      <xacro:property name="robot_rpy"    value="0 0 0"/>
+    </xacro:if>
+    <xacro:unless value="${base_at_world_origin}">
+      <xacro:property name="robot_parent" value="mount"/>
+      <xacro:property name="robot_xyz"    value="0 -0.218 0"/>
+      <xacro:property name="robot_rpy"    value="-1.5708 0 3.1416"/>
+    </xacro:unless>
+    <!-- ==================== UR3e Robot ==================== -->
+    <xacro:ur_robot
+      name="${ur_type}"
+      tf_prefix=""
+      parent="${robot_parent}"
+      joint_limits_parameters_file="$(find ur_description)/config/${ur_type}/joint_limits.yaml"
+      kinematics_parameters_file="$(find ur_description)/config/${ur_type}/default_kinematics.yaml"
+      physical_parameters_file="$(find ur_description)/config/${ur_type}/physical_parameters.yaml"
+      visual_parameters_file="$(find ur_description)/config/${ur_type}/visual_parameters.yaml"
+      transmission_hw_interface="hardware_interface/PositionJointInterface"
+      safety_limits="false"
+      safety_pos_margin="0.15"
+      safety_k_position="20"
+      use_mock_hardware="${use_mock_hardware}"
+      mock_sensor_commands="${mock_sensor_commands}"
+      headless_mode="${headless_mode}"
+      robot_ip="${robot_ip}"
+      script_filename="${script_filename}"
+      output_recipe_filename="${output_recipe_filename}"
+      input_recipe_filename="${input_recipe_filename}"
+      initial_positions_file="${initial_positions_file}"
+    >
+      <origin xyz="${robot_xyz}" rpy="${robot_rpy}"/>
+    </xacro:ur_robot>
+    <!-- ==================== Additional Elements (optional) ==================== -->
+    <!-- You can re-add monitor, wall, cameras, test plates etc. here,
+         by following the workstation pose conventions. -->
+  </xacro:macro>
 </robot>

Commit message: updated urdf collsion

File: TestSite/ws_rviz/src/ur3e_workstation/urdf/workstation.xacro (robot description, xacro)
@@ -102,5 +102,5 @@
         <mesh filename="package://ur3e_workstation/urdf/TestpladeKurve_v3.stl" scale="0.001 0.001 0.001"/>
       </geometry>
-      <origin xyz="0.200 0 0" rpy="1.5708 0 0"/>
+      <origin xyz="0.200 2.94 -0.4" rpy="1.5708 0 0"/>
     </collision>
   </link>

Commit message: should be functional

File: TestSite/ws_rviz/src/ur3e_workstation/urdf/workstation.xacro (robot description, xacro)
@@ -14,44 +14,4 @@
   <!-- ==================== World ==================== -->
   <link name="world"/>
-  <!-- ==================== Table / Bordplade ==================== -->
-  <link name="bordplade">
-    <visual>
-      <geometry>
-        <mesh filename="package://ur3e_workstation/urdf/Bundplade.stl" scale="0.001 0.001 0.001"/>
-      </geometry>
-      <origin xyz="0 0 0" rpy="0 0 0"/>
-    </visual>
-    <collision>
-      <geometry>
-        <mesh filename="package://ur3e_workstation/urdf/Bundplade.stl" scale="0.001 0.001 0.001"/>
-      </geometry>
-      <origin xyz="0 0 0" rpy="0 0 0"/>
-    </collision>
-  </link>
-  <joint name="world_to_bordplade" type="fixed">
-    <parent link="world"/>
-    <child link="bordplade"/>
-    <origin xyz="0 0 0" rpy="0 0 0"/>
-  </joint>
-  <!-- ==================== Mount ==================== -->
-  <link name="mount">
-    <visual>
-      <geometry>
-        <mesh filename="package://ur3e_workstation/urdf/UR3e_mount.stl" scale="0.001 0.001 0.001"/>
-      </geometry>
-      <origin xyz="0 0 0" rpy="0 0 0"/>
-    </visual>
-    <collision>
-      <geometry>
-        <mesh filename="package://ur3e_workstation/urdf/UR3e_mount.stl" scale="0.001 0.001 0.001"/>
-      </geometry>
-      <origin xyz="0 0 0" rpy="0 0 0"/>
-    </collision>
-  </link>
-  <joint name="bordplade_to_mount" type="fixed">
-    <parent link="bordplade"/>
-    <child link="mount"/>
-    <origin xyz="0.200 0.0 0.250" rpy="0 0 0"/>
-  </joint>
   <!-- ==================== UR3e Robot ==================== -->
   <xacro:include filename="$(find ur_description)/urdf/ur_macro.xacro"/>
@@ -63,6 +23,8 @@
   </xacro:if>
   <xacro:unless value="$(arg base_at_world_origin)">
-    <xacro:property name="robot_parent" value="mount"/>
-    <xacro:property name="robot_xyz" value="0 -0.218 0"/>
+    <!-- Robot attached to world at the mount position -->
+    <xacro:property name="robot_parent" value="world"/>
+    <!-- Mount pos (0.2, 0, 0.25) + Robot relative (0, -0.218, 0) -->
+    <xacro:property name="robot_xyz" value="0.2 -0.218 0.25"/>
     <xacro:property name="robot_rpy" value="-1.5708 0 3.1416"/>
   </xacro:unless>
@@ -90,24 +52,4 @@
     input_recipe_filename="$(arg input_recipe_filename)"
     kinematics_parameters_file="$(find ur_description)/config/$(arg ur_type)/default_kinematics.yaml"/>
-  <!-- ==================== Test Plate ==================== -->
-  <link name="testpladekurve">
-    <visual>
-      <geometry>
-        <mesh filename="package://ur3e_workstation/urdf/TestpladeKurve_v3.stl" scale="0.001 0.001 0.001"/>
-      </geometry>
-      <origin xyz="0.200 2.94 -0.4" rpy="1.5708 0 0"/>
-    </visual>
-    <collision>
-      <geometry>
-        <mesh filename="package://ur3e_workstation/urdf/TestpladeKurve_v3.stl" scale="0.001 0.001 0.001"/>
-      </geometry>
-      <origin xyz="0.200 2.94 -0.4" rpy="1.5708 0 0"/>
-    </collision>
-  </link>
-  <joint name="bordplade_to_testpladekurve" type="fixed">
-    <parent link="bordplade"/>
-    <child link="testpladekurve"/>
-    <origin xyz="0 0 0" rpy="0 0 0"/>
-  </joint>
   <!-- ==================== Realsense Holder ==================== -->
   <link name="realsense_holder">
